Commit message: Update go2_arx_badmiton.urdf
上一个修改只有重命名，没有修改里面的内容，现在加上

File: loco_manipulation_gym/resources/robots/go2_arx/urdf/go2_arx_badmiton.urdf (robot description, URDF)
Before this commit: robot go2_arx_description, 36 links, 35 joints
Links:
- added link badminton_racket, mass 0.1; collision mesh filename=../meshes/racket.STL scale=1 1 1; visual mesh filename=../meshes/racket.STL scale=1 1 1
Joints:
- added joint racket_fixed_joint: type fixed, parent arm_link6, child badminton_racket, origin xyz=0.05 0 0 rpy=0 1.5708 0
